File: test/test.kicad_pcb (KiCad board)
At the start: 2 copper layers, 173 parts, among them SW1 SW_Push, SW10 SW_Push, SW11 SW_Push, SW12 SW_Push, SW13 SW_Push, SW14 SW_Push, SW15 SW_Push, SW16 SW_Push, SW17 SW_Push, SW18 SW_Push, SW19 SW_Push, SW2 SW_Push, SW20 SW_Push, SW21 SW_Push, SW22 SW_Push, SW23 SW_Push, SW24 SW_Push, SW25 SW_Push, SW26 SW_Push, SW27 SW_Push, SW28 SW_Push, SW29 SW_Push, SW3 SW_Push, SW30 SW_Push, SW31 SW_Push, SW32 SW_Push, SW33 SW_Push, SW34 SW_Push, SW35 SW_Push, SW36 SW_Push, SW37 SW_Push, SW38 SW_Push, SW39 SW_Push, SW4 SW_Push, SW40 SW_Push, SW41 SW_Push, SW42 SW_Push, SW43 SW_Push, SW44 SW_Push, SW45 SW_Push, SW46 SW_Push, SW47 SW_Push, SW48 SW_Push, SW49 SW_Push, SW5 SW_Push, SW50 SW_Push, SW51 SW_Push, SW52 SW_Push, SW53 SW_Push, SW54 SW_Push, SW55 SW_Push, SW56 SW_Push, SW57 SW_Push, SW58 SW_Push, SW59 SW_Push, SW6 SW_Push, SW60 SW_Push, SW61 SW_Push, SW62 SW_Push, SW63 SW_Push, SW64 SW_Push, SW65 SW_Push, SW66 SW_Push, SW67 SW_Push, SW68 SW_Push, SW69 SW_Push, SW7 SW_Push, SW70 SW_Push, SW71 SW_Push, SW72 SW_Push, SW73 SW_Push, SW74 SW_Push, SW75 SW_Push, SW76 SW_Push, SW77 SW_Push, SW78 SW_Push, SW79 SW_Push, SW8 SW_Push, SW80 SW_Push, SW81 SW_Push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

Commit message: Finished the pcb design
Parts:
- moved D15 270.5 mm to (317.6, 51.7)
- moved SW15 270.5 mm to (312.6, 47.7)
- moved D82 265.3 mm to (298.6, 147.0)
- moved SW82 265.3 mm to (293.5, 143.0)
- moved S2 262.1 mm to (300.7, 104.9)
- moved SW73 235.9 mm to (312.6, 123.9)
- moved D73 235.9 mm to (317.6, 127.9)
- moved D49 227.6 mm to (103.3, 108.9)
- moved SW49 227.6 mm to (98.3, 104.9)
- moved S3 227.1 mm to (57.8, 123.9)
- moved SW34 208.1 mm to (93.5, 85.8)
- moved D34 208.1 mm to (98.6, 89.8)
- moved D80 206.3 mm to (246.2, 147.0)
- moved SW80 206.3 mm to (241.1, 143.0)
- moved SW76 200.5 mm to (72.1, 143.0)
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Connections:
- A1 pad 1: /Row1 -> /Col1
- A1 pad 10: /Col2 -> /Col8
- A1 pad 11: /Col3 -> /Col9
- A1 pad 12: /Col4 -> /Col10
- A1 pad 14: /Col5 -> /Col11
- A1 pad 15: /Col6 -> /Col12
- A1 pad 16: /Col7 -> /Col13
- A1 pad 17: /Col8 -> /Col14
- A1 pad 19: /Col9 -> /Col15
- A1 pad 2: /Row2 -> /Col2
- A1 pad 20: /Col10 -> /Col16
- A1 pad 21: /Col11 -> unconnected-(A1-GPIO16-Pad21)
- A1 pad 22: /Col12 -> /Row1
- A1 pad 24: /Col13 -> /Row2
- A1 pad 25: /Col14 -> /Row3
- A1 pad 26: /Col15 -> /Row4
- A1 pad 27: /Col16 -> /Row5
- A1 pad 29: unconnected-(A1-GPIO22-Pad29) -> /Row6
- A1 pad 4: /Row3 -> /Col3
- A1 pad 5: /Row4 -> /Col4
- A1 pad 6: /Row5 -> /Col5
- A1 pad 7: /Row6 -> /Col6
- A1 pad 9: /Col1 -> /Col7
- SW79 pad 1: /Col10 -> /Col9
- SW80 pad 1: /Col11 -> /Col10
- SW81 pad 1: /Col12 -> /Col11
Routing:
- net /Col1: track 0.00 -> 408.7 mm
- net /Col2: track 0.00 -> 398.6 mm
- net /Col3: track 0.00 -> 380.7 mm
- net /Row6: track 0.00 -> 376.1 mm
- net /Row1: track 0.00 -> 351.0 mm
- net /Row5: track 0.00 -> 342.1 mm
- net /Col4: track 0.00 -> 338.9 mm
- net /Row2: track 0.00 -> 338.4 mm
- net /Row4: track 0.00 -> 329.7 mm
- net /Col6: track 0.00 -> 321.6 mm, vias 0 -> 2
- net /Row3: track 0.00 -> 321.6 mm
- net /Col5: track 0.00 -> 319.1 mm, vias 0 -> 2
- net /Col7: track 0.00 -> 284.6 mm, vias 0 -> 2
- net /Col9: track 0.00 -> 268.6 mm, vias 0 -> 2
- net /Col8: track 0.00 -> 267.1 mm, vias 0 -> 2
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- added copper zone on B.Cu, net GND
- added copper zone on F.Cu, net GND
Other:
- board outline added: 331.8 x 116.7 mm
