File: keyboard-full/untitled.kicad_sch (KiCad schematic)
At the start: 0 parts

Commit message: redid the keyboard pcb design
Parts:
- added D92: SK6812MINI-E, LED_SMD:LED_SK6812MINI-E_3.2x2.8mm_P1.5mm_ReverseMount, symbol LED:SK6812MINI-E
- added U1, U2, U3: IS31FL3736, Package_DFN_QFN:QFN-40-1EP_5x5mm_P0.4mm_EP3.8x3.8mm, symbol Driver_LED:IS31FL3736
Connections:
- new net: U1.11 (PGND), U1.4 (PGND)
- new net: U1.40 (GND), U1.41 (GND)
- new net: U3.11 (PGND), U3.4 (PGND)
- new net: U3.40 (GND), U3.41 (GND)
- new net: U2.11 (PGND), U2.4 (PGND)
- new net: U2.40 (GND), U2.41 (GND)

Commit message: Fixes to schema
Parts:
- removed D92: SK6812MINI-E, LED_SMD:LED_SK6812MINI-E_3.2x2.8mm_P1.5mm_ReverseMount, symbol LED:SK6812MINI-E
- removed U1, U2, U3: IS31FL3736, Package_DFN_QFN:QFN-40-1EP_5x5mm_P0.4mm_EP3.8x3.8mm, symbol Driver_LED:IS31FL3736
