File: keyboard-full/keyboard-full.kicad_pcb (KiCad board)
At the start: 2 copper layers, 184 parts, among them SW1 SW_Push, SW10 SW_Push, SW11 SW_Push, SW12 SW_Push, SW13 SW_Push, SW14 SW_Push, SW15 SW_Push, SW16 SW_Push, SW17 SW_Push, SW18 SW_Push, SW19 SW_Push, SW2 SW_Push, SW20 SW_Push, SW21 SW_Push, SW22 SW_Push, SW23 SW_Push, SW24 SW_Push, SW25 SW_Push, SW26 SW_Push, SW27 SW_Push, SW28 SW_Push, SW29 SW_Push, SW3 SW_Push, SW30 SW_Push, SW31 SW_Push, SW32 SW_Push, SW33 SW_Push, SW34 SW_Push, SW35 SW_Push, SW36 SW_Push, SW37 SW_Push, SW38 SW_Push, SW39 SW_Push, SW4 SW_Push, SW40 SW_Push, SW41 SW_Push, SW42 SW_Push, SW43 SW_Push, SW44 SW_Push, SW45 SW_Push, SW46 SW_Push, SW47 SW_Push, SW48 SW_Push, SW49 SW_Push, SW5 SW_Push, SW50 SW_Push, SW51 SW_Push, SW52 SW_Push, SW53 SW_Push, SW54 SW_Push, SW55 SW_Push, SW56 SW_Push, SW57 SW_Push, SW58 SW_Push, SW59 SW_Push, SW6 SW_Push, SW60 SW_Push, SW61 SW_Push, SW62 SW_Push, SW63 SW_Push, SW64 SW_Push, SW65 SW_Push, SW66 SW_Push, SW67 SW_Push, SW68 SW_Push, SW69 SW_Push, SW7 SW_Push, SW70 SW_Push, SW71 SW_Push, SW72 SW_Push, SW73 SW_Push, SW74 SW_Push, SW75 SW_Push, SW76 SW_Push, SW77 SW_Push, SW78 SW_Push, SW79 SW_Push, SW8 SW_Push, SW80 SW_Push, SW81 SW_Push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

Commit message: progress on keyboard
Parts:
- removed SW1, SW10, SW11, SW12, SW13, SW14, SW15, SW16, SW17, SW18, SW19, SW2, SW20, SW21, SW22, SW23, SW24, SW25, SW26, SW27, SW28, SW29, SW3, SW30, SW31, SW32, SW33, SW34, SW35, SW36, SW37, SW38, SW39, SW4, SW40, SW41, SW42, SW43, SW44, SW45, SW46, SW47, SW48, SW49, SW5, SW50, SW51, SW52, SW53, SW54, SW55, SW56, SW57, SW58, SW59, SW6, SW60, SW61, SW62, SW63, SW64, SW65, SW66, SW67, SW68, SW69, SW7, SW70, SW71, SW72, SW73, SW74, SW75, SW76, SW77, SW78, SW79, SW8, SW80, SW81, SW82, SW83 (x2), SW85, SW86, SW87, SW88, SW89, SW9, SW90, SW91: SW_Push, PCM_marbastlib-mx:SW_MX_1u
- removed SW84: SW_Push, PCM_marbastlib-mx:STAB_MX_P_6u
- added C1: 0.1uF, Capacitor_SMD:C_1206_3216Metric_Pad1.33x1.80mm_HandSolder, B.Cu at (38.1, 46.1)
- added C10: 0.1uF, Capacitor_SMD:C_1206_3216Metric_Pad1.33x1.80mm_HandSolder, B.Cu at (247.7, 46.1)
- added C11: 0.1uF, Capacitor_SMD:C_1206_3216Metric_Pad1.33x1.80mm_HandSolder, B.Cu at (266.7, 46.1)
- added C12: 0.1uF, Capacitor_SMD:C_1206_3216Metric_Pad1.33x1.80mm_HandSolder, B.Cu at (285.8, 46.1)
- added C13: 0.1uF, Capacitor_SMD:C_1206_3216Metric_Pad1.33x1.80mm_HandSolder, B.Cu at (304.8, 46.1)
- added C14: 0.1uF, Capacitor_SMD:C_1206_3216Metric_Pad1.33x1.80mm_HandSolder, B.Cu at (347.7, 46.1)
- added C15: 0.1uF, Capacitor_SMD:C_1206_3216Metric_Pad1.33x1.80mm_HandSolder, B.Cu at (366.7, 46.1)
- added C16: 0.1uF, Capacitor_SMD:C_1206_3216Metric_Pad1.33x1.80mm_HandSolder, B.Cu at (385.8, 46.1)
- added C17: 0.1uF, Capacitor_SMD:C_1206_3216Metric_Pad1.33x1.80mm_HandSolder, B.Cu at (38.1, 74.7)
- added C18: 0.1uF, Capacitor_SMD:C_1206_3216Metric_Pad1.33x1.80mm_HandSolder, B.Cu at (57.1, 74.7)
- added C19: 0.1uF, Capacitor_SMD:C_1206_3216Metric_Pad1.33x1.80mm_HandSolder, B.Cu at (76.2, 74.7)
- added C2: 0.1uF, Capacitor_SMD:C_1206_3216Metric_Pad1.33x1.80mm_HandSolder, B.Cu at (76.2, 46.1)
- added C20: 0.1uF, Capacitor_SMD:C_1206_3216Metric_Pad1.33x1.80mm_HandSolder, B.Cu at (95.2, 74.7)
- added C21: 0.1uF, Capacitor_SMD:C_1206_3216Metric_Pad1.33x1.80mm_HandSolder, B.Cu at (114.3, 74.7)
- added C22: 0.1uF, Capacitor_SMD:C_1206_3216Metric_Pad1.33x1.80mm_HandSolder, B.Cu at (133.3, 74.7)
- added C23: 0.1uF, Capacitor_SMD:C_1206_3216Metric_Pad1.33x1.80mm_HandSolder, B.Cu at (152.4, 74.7)
- added C24: 0.1uF, Capacitor_SMD:C_1206_3216Metric_Pad1.33x1.80mm_HandSolder, B.Cu at (171.4, 74.7)
- added C25: 0.1uF, Capacitor_SMD:C_1206_3216Metric_Pad1.33x1.80mm_HandSolder, B.Cu at (190.5, 74.7)
- added C26: 0.1uF, Capacitor_SMD:C_1206_3216Metric_Pad1.33x1.80mm_HandSolder, B.Cu at (209.6, 74.7)
- added C27: 0.1uF, Capacitor_SMD:C_1206_3216Metric_Pad1.33x1.80mm_HandSolder, B.Cu at (228.6, 74.7)
- added C28: 0.1uF, Capacitor_SMD:C_1206_3216Metric_Pad1.33x1.80mm_HandSolder, B.Cu at (247.7, 74.7)
- added C29: 0.1uF, Capacitor_SMD:C_1206_3216Metric_Pad1.33x1.80mm_HandSolder, B.Cu at (266.7, 74.7)
- added C3: 0.1uF, Capacitor_SMD:C_1206_3216Metric_Pad1.33x1.80mm_HandSolder, B.Cu at (95.2, 46.1)
- added C30: 0.1uF, Capacitor_SMD:C_1206_3216Metric_Pad1.33x1.80mm_HandSolder, B.Cu at (295.3, 74.7)
- added C31: 0.1uF, Capacitor_SMD:C_1206_3216Metric_Pad1.33x1.80mm_HandSolder, B.Cu at (347.7, 74.7)
- added C32: 0.1uF, Capacitor_SMD:C_1206_3216Metric_Pad1.33x1.80mm_HandSolder, B.Cu at (366.7, 74.7)
- added C33: 0.1uF, Capacitor_SMD:C_1206_3216Metric_Pad1.33x1.80mm_HandSolder, B.Cu at (385.8, 74.7)
- added C34: 0.1uF, Capacitor_SMD:C_1206_3216Metric_Pad1.33x1.80mm_HandSolder, B.Cu at (42.9, 93.7)
- added C35: 0.1uF, Capacitor_SMD:C_1206_3216Metric_Pad1.33x1.80mm_HandSolder, B.Cu at (66.7, 93.7)
- added C36: 0.1uF, Capacitor_SMD:C_1206_3216Metric_Pad1.33x1.80mm_HandSolder, B.Cu at (85.7, 93.7)
- added C37: 0.1uF, Capacitor_SMD:C_1206_3216Metric_Pad1.33x1.80mm_HandSolder, B.Cu at (104.8, 93.7)
- added C38: 0.1uF, Capacitor_SMD:C_1206_3216Metric_Pad1.33x1.80mm_HandSolder, B.Cu at (123.8, 93.7)
- added C39: 0.1uF, Capacitor_SMD:C_1206_3216Metric_Pad1.33x1.80mm_HandSolder, B.Cu at (142.9, 93.7)
- added C4: 0.1uF, Capacitor_SMD:C_1206_3216Metric_Pad1.33x1.80mm_HandSolder, B.Cu at (114.3, 46.1)
- added C40: 0.1uF, Capacitor_SMD:C_1206_3216Metric_Pad1.33x1.80mm_HandSolder, B.Cu at (161.9, 93.7)
- added C41: 0.1uF, Capacitor_SMD:C_1206_3216Metric_Pad1.33x1.80mm_HandSolder, B.Cu at (181.0, 93.7)
- added C42: 0.1uF, Capacitor_SMD:C_1206_3216Metric_Pad1.33x1.80mm_HandSolder, B.Cu at (200.0, 93.7)
- added C43: 0.1uF, Capacitor_SMD:C_1206_3216Metric_Pad1.33x1.80mm_HandSolder, B.Cu at (219.1, 93.7)
- added C44: 0.1uF, Capacitor_SMD:C_1206_3216Metric_Pad1.33x1.80mm_HandSolder, B.Cu at (238.1, 93.7)
- added C45: 0.1uF, Capacitor_SMD:C_1206_3216Metric_Pad1.33x1.80mm_HandSolder, B.Cu at (257.2, 93.7)
- added C46: 0.1uF, Capacitor_SMD:C_1206_3216Metric_Pad1.33x1.80mm_HandSolder, B.Cu at (276.2, 93.7)
- added C47: 0.1uF, Capacitor_SMD:C_1206_3216Metric_Pad1.33x1.80mm_HandSolder, B.Cu at (300.0, 93.7)
- added C48: 0.1uF, Capacitor_SMD:C_1206_3216Metric_Pad1.33x1.80mm_HandSolder, B.Cu at (347.7, 93.7)
- added C49: 0.1uF, Capacitor_SMD:C_1206_3216Metric_Pad1.33x1.80mm_HandSolder, B.Cu at (366.7, 93.7)
- added C5: 0.1uF, Capacitor_SMD:C_1206_3216Metric_Pad1.33x1.80mm_HandSolder, B.Cu at (133.3, 46.1)
- added C50: 0.1uF, Capacitor_SMD:C_1206_3216Metric_Pad1.33x1.80mm_HandSolder, B.Cu at (385.8, 93.7)
- added C51: 0.1uF, Capacitor_SMD:C_1206_3216Metric_Pad1.33x1.80mm_HandSolder, B.Cu at (45.2, 112.8)
- added C52: 0.1uF, Capacitor_SMD:C_1206_3216Metric_Pad1.33x1.80mm_HandSolder, B.Cu at (71.4, 112.8)
- added C53: 0.1uF, Capacitor_SMD:C_1206_3216Metric_Pad1.33x1.80mm_HandSolder, B.Cu at (90.5, 112.8)
- added C54: 0.1uF, Capacitor_SMD:C_1206_3216Metric_Pad1.33x1.80mm_HandSolder, B.Cu at (109.5, 112.8)
- added C55: 0.1uF, Capacitor_SMD:C_1206_3216Metric_Pad1.33x1.80mm_HandSolder, B.Cu at (128.6, 112.8)
- added C56: 0.1uF, Capacitor_SMD:C_1206_3216Metric_Pad1.33x1.80mm_HandSolder, B.Cu at (147.6, 112.8)
- added C57: 0.1uF, Capacitor_SMD:C_1206_3216Metric_Pad1.33x1.80mm_HandSolder, B.Cu at (166.7, 112.8)
- added C58: 0.1uF, Capacitor_SMD:C_1206_3216Metric_Pad1.33x1.80mm_HandSolder, B.Cu at (185.7, 112.8)
- added C59: 0.1uF, Capacitor_SMD:C_1206_3216Metric_Pad1.33x1.80mm_HandSolder, B.Cu at (204.8, 112.8)
- added C6: 0.1uF, Capacitor_SMD:C_1206_3216Metric_Pad1.33x1.80mm_HandSolder, B.Cu at (161.9, 46.1)
- added C60: 0.1uF, Capacitor_SMD:C_1206_3216Metric_Pad1.33x1.80mm_HandSolder, B.Cu at (223.8, 112.8)
- added C61: 0.1uF, Capacitor_SMD:C_1206_3216Metric_Pad1.33x1.80mm_HandSolder, B.Cu at (242.9, 112.8)
- added C62: 0.1uF, Capacitor_SMD:C_1206_3216Metric_Pad1.33x1.80mm_HandSolder, B.Cu at (261.9, 112.8)
- added C63: 0.1uF, Capacitor_SMD:C_1206_3216Metric_Pad1.33x1.80mm_HandSolder, B.Cu at (292.9, 112.8)
- added C64: 0.1uF, Capacitor_SMD:C_1206_3216Metric_Pad1.33x1.80mm_HandSolder, B.Cu at (47.6, 131.8)
- added C65: 0.1uF, Capacitor_SMD:C_1206_3216Metric_Pad1.33x1.80mm_HandSolder, B.Cu at (76.2, 131.8)
- added C66: 0.1uF, Capacitor_SMD:C_1206_3216Metric_Pad1.33x1.80mm_HandSolder, B.Cu at (95.2, 131.8)
- added C67: 0.1uF, Capacitor_SMD:C_1206_3216Metric_Pad1.33x1.80mm_HandSolder, B.Cu at (114.3, 131.8)
- added C68: 0.1uF, Capacitor_SMD:C_1206_3216Metric_Pad1.33x1.80mm_HandSolder, B.Cu at (133.3, 131.8)
- added C69: 0.1uF, Capacitor_SMD:C_1206_3216Metric_Pad1.33x1.80mm_HandSolder, B.Cu at (152.4, 131.8)
- added C7: 0.1uF, Capacitor_SMD:C_1206_3216Metric_Pad1.33x1.80mm_HandSolder, B.Cu at (181.0, 46.1)
- added C70: 0.1uF, Capacitor_SMD:C_1206_3216Metric_Pad1.33x1.80mm_HandSolder, B.Cu at (171.4, 131.8)
- added C71: 0.1uF, Capacitor_SMD:C_1206_3216Metric_Pad1.33x1.80mm_HandSolder, B.Cu at (190.5, 131.8)
- added C72: 0.1uF, Capacitor_SMD:C_1206_3216Metric_Pad1.33x1.80mm_HandSolder, B.Cu at (209.6, 131.8)
- added C73: 0.1uF, Capacitor_SMD:C_1206_3216Metric_Pad1.33x1.80mm_HandSolder, B.Cu at (228.6, 131.8)
- added C74: 0.1uF, Capacitor_SMD:C_1206_3216Metric_Pad1.33x1.80mm_HandSolder, B.Cu at (247.7, 131.8)
- added C75: 0.1uF, Capacitor_SMD:C_1206_3216Metric_Pad1.33x1.80mm_HandSolder, B.Cu at (266.7, 131.8)
- added C76: 0.1uF, Capacitor_SMD:C_1206_3216Metric_Pad1.33x1.80mm_HandSolder, B.Cu at (285.8, 131.8)
- added C77: 0.1uF, Capacitor_SMD:C_1206_3216Metric_Pad1.33x1.80mm_HandSolder, B.Cu at (304.8, 131.8)
- added C78: 0.1uF, Capacitor_SMD:C_1206_3216Metric_Pad1.33x1.80mm_HandSolder, B.Cu at (347.7, 131.8)
- added C79: 0.1uF, Capacitor_SMD:C_1206_3216Metric_Pad1.33x1.80mm_HandSolder, B.Cu at (366.7, 131.8)
- added C8: 0.1uF, Capacitor_SMD:C_1206_3216Metric_Pad1.33x1.80mm_HandSolder, B.Cu at (200.0, 46.1)
- added C80: 0.1uF, Capacitor_SMD:C_1206_3216Metric_Pad1.33x1.80mm_HandSolder, B.Cu at (385.8, 131.8)
- added C81: 0.1uF, Capacitor_SMD:C_1206_3216Metric_Pad1.33x1.80mm_HandSolder, B.Cu at (40.5, 150.9)
- added C82: 0.1uF, Capacitor_SMD:C_1206_3216Metric_Pad1.33x1.80mm_HandSolder, B.Cu at (64.3, 150.9)
- added C83: 0.1uF, Capacitor_SMD:C_1206_3216Metric_Pad1.33x1.80mm_HandSolder, B.Cu at (88.1, 150.9)
- added C84: 0.1uF, Capacitor_SMD:C_1206_3216Metric_Pad1.33x1.80mm_HandSolder, B.Cu at (159.5, 150.9)
- added C85: 0.1uF, Capacitor_SMD:C_1206_3216Metric_Pad1.33x1.80mm_HandSolder, B.Cu at (231.0, 150.9)
- added C86: 0.1uF, Capacitor_SMD:C_1206_3216Metric_Pad1.33x1.80mm_HandSolder, B.Cu at (254.8, 150.9)
- added C87: 0.1uF, Capacitor_SMD:C_1206_3216Metric_Pad1.33x1.80mm_HandSolder, B.Cu at (278.6, 150.9)
- added C88: 0.1uF, Capacitor_SMD:C_1206_3216Metric_Pad1.33x1.80mm_HandSolder, B.Cu at (302.4, 150.9)
- added C89: 0.1uF, Capacitor_SMD:C_1206_3216Metric_Pad1.33x1.80mm_HandSolder, B.Cu at (347.7, 150.9)
- added C9: 0.1uF, Capacitor_SMD:C_1206_3216Metric_Pad1.33x1.80mm_HandSolder, B.Cu at (219.1, 46.1)
- added C90: 0.1uF, Capacitor_SMD:C_1206_3216Metric_Pad1.33x1.80mm_HandSolder, B.Cu at (366.7, 150.9)
- added C91: 0.1uF, Capacitor_SMD:C_1206_3216Metric_Pad1.33x1.80mm_HandSolder, B.Cu at (385.8, 150.9)
- added H1: MountingHole, MountingHole:MountingHole_2.1mm, F.Cu at (237.3, 250.8)
- added H2: MountingHole, MountingHole:MountingHole_2.1mm, F.Cu at (242.1, 250.8)
- added H3: MountingHole, MountingHole:MountingHole_2.1mm, F.Cu at (246.8, 250.8)
- added H4: MountingHole, MountingHole:MountingHole_2.1mm, F.Cu at (251.6, 250.8)
- added LED1: SK6812MINI-E, LED_SMD:LED_SK6812MINI-E_3.2x2.8mm_P1.5mm_ReverseMount, B.Cu at (38.1, 43.1)
- added LED10: SK6812MINI-E, LED_SMD:LED_SK6812MINI-E_3.2x2.8mm_P1.5mm_ReverseMount, B.Cu at (247.7, 43.1)
- added LED11: SK6812MINI-E, LED_SMD:LED_SK6812MINI-E_3.2x2.8mm_P1.5mm_ReverseMount, B.Cu at (266.7, 43.1)
- added LED12: SK6812MINI-E, LED_SMD:LED_SK6812MINI-E_3.2x2.8mm_P1.5mm_ReverseMount, B.Cu at (285.8, 43.1)
- added LED13: SK6812MINI-E, LED_SMD:LED_SK6812MINI-E_3.2x2.8mm_P1.5mm_ReverseMount, B.Cu at (304.8, 43.1)
- added LED14: SK6812MINI-E, LED_SMD:LED_SK6812MINI-E_3.2x2.8mm_P1.5mm_ReverseMount, B.Cu at (347.7, 43.1)
- added LED15: SK6812MINI-E, LED_SMD:LED_SK6812MINI-E_3.2x2.8mm_P1.5mm_ReverseMount, B.Cu at (366.7, 43.1)
- added LED16: SK6812MINI-E, LED_SMD:LED_SK6812MINI-E_3.2x2.8mm_P1.5mm_ReverseMount, B.Cu at (385.8, 43.1)
- added LED17: SK6812MINI-E, LED_SMD:LED_SK6812MINI-E_3.2x2.8mm_P1.5mm_ReverseMount, B.Cu at (38.1, 71.7)
- added LED18: SK6812MINI-E, LED_SMD:LED_SK6812MINI-E_3.2x2.8mm_P1.5mm_ReverseMount, B.Cu at (57.1, 71.7)
- added LED19: SK6812MINI-E, LED_SMD:LED_SK6812MINI-E_3.2x2.8mm_P1.5mm_ReverseMount, B.Cu at (76.2, 71.7)
- added LED2: SK6812MINI-E, LED_SMD:LED_SK6812MINI-E_3.2x2.8mm_P1.5mm_ReverseMount, B.Cu at (76.2, 43.1)
- added LED20: SK6812MINI-E, LED_SMD:LED_SK6812MINI-E_3.2x2.8mm_P1.5mm_ReverseMount, B.Cu at (95.2, 71.7)
- added LED21: SK6812MINI-E, LED_SMD:LED_SK6812MINI-E_3.2x2.8mm_P1.5mm_ReverseMount, B.Cu at (114.3, 71.7)
- added LED22: SK6812MINI-E, LED_SMD:LED_SK6812MINI-E_3.2x2.8mm_P1.5mm_ReverseMount, B.Cu at (133.3, 71.7)
- added LED23: SK6812MINI-E, LED_SMD:LED_SK6812MINI-E_3.2x2.8mm_P1.5mm_ReverseMount, B.Cu at (152.4, 71.7)
- added LED24: SK6812MINI-E, LED_SMD:LED_SK6812MINI-E_3.2x2.8mm_P1.5mm_ReverseMount, B.Cu at (171.4, 71.7)
- added LED25: SK6812MINI-E, LED_SMD:LED_SK6812MINI-E_3.2x2.8mm_P1.5mm_ReverseMount, B.Cu at (190.5, 71.7)
- added LED26: SK6812MINI-E, LED_SMD:LED_SK6812MINI-E_3.2x2.8mm_P1.5mm_ReverseMount, B.Cu at (209.6, 71.7)
- added LED27: SK6812MINI-E, LED_SMD:LED_SK6812MINI-E_3.2x2.8mm_P1.5mm_ReverseMount, B.Cu at (228.6, 71.7)
- added LED28: SK6812MINI-E, LED_SMD:LED_SK6812MINI-E_3.2x2.8mm_P1.5mm_ReverseMount, B.Cu at (247.7, 71.7)
- added LED29: SK6812MINI-E, LED_SMD:LED_SK6812MINI-E_3.2x2.8mm_P1.5mm_ReverseMount, B.Cu at (266.7, 71.7)
- added LED3: SK6812MINI-E, LED_SMD:LED_SK6812MINI-E_3.2x2.8mm_P1.5mm_ReverseMount, B.Cu at (95.2, 43.1)
- added LED30: SK6812MINI-E, LED_SMD:LED_SK6812MINI-E_3.2x2.8mm_P1.5mm_ReverseMount, B.Cu at (295.3, 71.7)
- added LED31: SK6812MINI-E, LED_SMD:LED_SK6812MINI-E_3.2x2.8mm_P1.5mm_ReverseMount, B.Cu at (347.7, 71.7)
- added LED32: SK6812MINI-E, LED_SMD:LED_SK6812MINI-E_3.2x2.8mm_P1.5mm_ReverseMount, B.Cu at (366.7, 71.7)
- added LED33: SK6812MINI-E, LED_SMD:LED_SK6812MINI-E_3.2x2.8mm_P1.5mm_ReverseMount, B.Cu at (385.8, 71.7)
- added LED34: SK6812MINI-E, LED_SMD:LED_SK6812MINI-E_3.2x2.8mm_P1.5mm_ReverseMount, B.Cu at (42.9, 90.7)
- added LED35: SK6812MINI-E, LED_SMD:LED_SK6812MINI-E_3.2x2.8mm_P1.5mm_ReverseMount, B.Cu at (66.7, 90.7)
- added LED36: SK6812MINI-E, LED_SMD:LED_SK6812MINI-E_3.2x2.8mm_P1.5mm_ReverseMount, B.Cu at (85.7, 90.7)
- added LED37: SK6812MINI-E, LED_SMD:LED_SK6812MINI-E_3.2x2.8mm_P1.5mm_ReverseMount, B.Cu at (104.8, 90.7)
- added LED38: SK6812MINI-E, LED_SMD:LED_SK6812MINI-E_3.2x2.8mm_P1.5mm_ReverseMount, B.Cu at (123.8, 90.7)
- added LED39: SK6812MINI-E, LED_SMD:LED_SK6812MINI-E_3.2x2.8mm_P1.5mm_ReverseMount, B.Cu at (142.9, 90.7)
- added LED4: SK6812MINI-E, LED_SMD:LED_SK6812MINI-E_3.2x2.8mm_P1.5mm_ReverseMount, B.Cu at (114.3, 43.1)
- added LED40: SK6812MINI-E, LED_SMD:LED_SK6812MINI-E_3.2x2.8mm_P1.5mm_ReverseMount, B.Cu at (161.9, 90.7)
- added LED41: SK6812MINI-E, LED_SMD:LED_SK6812MINI-E_3.2x2.8mm_P1.5mm_ReverseMount, B.Cu at (181.0, 90.7)
- added LED42: SK6812MINI-E, LED_SMD:LED_SK6812MINI-E_3.2x2.8mm_P1.5mm_ReverseMount, B.Cu at (200.0, 90.7)
- added LED43: SK6812MINI-E, LED_SMD:LED_SK6812MINI-E_3.2x2.8mm_P1.5mm_ReverseMount, B.Cu at (219.1, 90.7)
- added LED44: SK6812MINI-E, LED_SMD:LED_SK6812MINI-E_3.2x2.8mm_P1.5mm_ReverseMount, B.Cu at (238.1, 90.7)
- added LED45: SK6812MINI-E, LED_SMD:LED_SK6812MINI-E_3.2x2.8mm_P1.5mm_ReverseMount, B.Cu at (257.2, 90.7)
- added LED46: SK6812MINI-E, LED_SMD:LED_SK6812MINI-E_3.2x2.8mm_P1.5mm_ReverseMount, B.Cu at (276.2, 90.7)
- added LED47: SK6812MINI-E, LED_SMD:LED_SK6812MINI-E_3.2x2.8mm_P1.5mm_ReverseMount, B.Cu at (300.0, 90.7)
- added LED48: SK6812MINI-E, LED_SMD:LED_SK6812MINI-E_3.2x2.8mm_P1.5mm_ReverseMount, B.Cu at (347.7, 90.7)
- added LED49: SK6812MINI-E, LED_SMD:LED_SK6812MINI-E_3.2x2.8mm_P1.5mm_ReverseMount, B.Cu at (366.7, 90.7)
- added LED5: SK6812MINI-E, LED_SMD:LED_SK6812MINI-E_3.2x2.8mm_P1.5mm_ReverseMount, B.Cu at (133.3, 43.1)
- added LED50: SK6812MINI-E, LED_SMD:LED_SK6812MINI-E_3.2x2.8mm_P1.5mm_ReverseMount, B.Cu at (385.8, 90.7)
- added LED51: SK6812MINI-E, LED_SMD:LED_SK6812MINI-E_3.2x2.8mm_P1.5mm_ReverseMount, B.Cu at (45.2, 109.8)
- added LED52: SK6812MINI-E, LED_SMD:LED_SK6812MINI-E_3.2x2.8mm_P1.5mm_ReverseMount, B.Cu at (71.4, 109.8)
- added LED53: SK6812MINI-E, LED_SMD:LED_SK6812MINI-E_3.2x2.8mm_P1.5mm_ReverseMount, B.Cu at (90.5, 109.8)
- added LED54: SK6812MINI-E, LED_SMD:LED_SK6812MINI-E_3.2x2.8mm_P1.5mm_ReverseMount, B.Cu at (109.5, 109.8)
- added LED55: SK6812MINI-E, LED_SMD:LED_SK6812MINI-E_3.2x2.8mm_P1.5mm_ReverseMount, B.Cu at (128.6, 109.8)
- added LED56: SK6812MINI-E, LED_SMD:LED_SK6812MINI-E_3.2x2.8mm_P1.5mm_ReverseMount, B.Cu at (147.6, 109.8)
- added LED57: SK6812MINI-E, LED_SMD:LED_SK6812MINI-E_3.2x2.8mm_P1.5mm_ReverseMount, B.Cu at (166.7, 109.8)
- added LED58: SK6812MINI-E, LED_SMD:LED_SK6812MINI-E_3.2x2.8mm_P1.5mm_ReverseMount, B.Cu at (185.7, 109.8)
- added LED59: SK6812MINI-E, LED_SMD:LED_SK6812MINI-E_3.2x2.8mm_P1.5mm_ReverseMount, B.Cu at (204.8, 109.8)
- added LED6: SK6812MINI-E, LED_SMD:LED_SK6812MINI-E_3.2x2.8mm_P1.5mm_ReverseMount, B.Cu at (161.9, 43.1)
- added LED60: SK6812MINI-E, LED_SMD:LED_SK6812MINI-E_3.2x2.8mm_P1.5mm_ReverseMount, B.Cu at (223.8, 109.8)
- added LED61: SK6812MINI-E, LED_SMD:LED_SK6812MINI-E_3.2x2.8mm_P1.5mm_ReverseMount, B.Cu at (242.9, 109.8)
- added LED62: SK6812MINI-E, LED_SMD:LED_SK6812MINI-E_3.2x2.8mm_P1.5mm_ReverseMount, B.Cu at (261.9, 109.8)
- added LED63: SK6812MINI-E, LED_SMD:LED_SK6812MINI-E_3.2x2.8mm_P1.5mm_ReverseMount, B.Cu at (292.9, 109.8)
- added LED64: SK6812MINI-E, LED_SMD:LED_SK6812MINI-E_3.2x2.8mm_P1.5mm_ReverseMount, B.Cu at (47.6, 128.8)
- added LED65: SK6812MINI-E, LED_SMD:LED_SK6812MINI-E_3.2x2.8mm_P1.5mm_ReverseMount, B.Cu at (76.2, 128.8)
- added LED66: SK6812MINI-E, LED_SMD:LED_SK6812MINI-E_3.2x2.8mm_P1.5mm_ReverseMount, B.Cu at (95.2, 128.8)
- added LED67: SK6812MINI-E, LED_SMD:LED_SK6812MINI-E_3.2x2.8mm_P1.5mm_ReverseMount, B.Cu at (114.3, 128.8)
- added LED68: SK6812MINI-E, LED_SMD:LED_SK6812MINI-E_3.2x2.8mm_P1.5mm_ReverseMount, B.Cu at (133.3, 128.8)
- added LED69: SK6812MINI-E, LED_SMD:LED_SK6812MINI-E_3.2x2.8mm_P1.5mm_ReverseMount, B.Cu at (152.4, 128.8)
- added LED7: SK6812MINI-E, LED_SMD:LED_SK6812MINI-E_3.2x2.8mm_P1.5mm_ReverseMount, B.Cu at (181.0, 43.1)
- added LED70: SK6812MINI-E, LED_SMD:LED_SK6812MINI-E_3.2x2.8mm_P1.5mm_ReverseMount, B.Cu at (171.4, 128.8)
- added LED71: SK6812MINI-E, LED_SMD:LED_SK6812MINI-E_3.2x2.8mm_P1.5mm_ReverseMount, B.Cu at (190.5, 128.8)
- added LED72: SK6812MINI-E, LED_SMD:LED_SK6812MINI-E_3.2x2.8mm_P1.5mm_ReverseMount, B.Cu at (209.6, 128.8)
- added LED73: SK6812MINI-E, LED_SMD:LED_SK6812MINI-E_3.2x2.8mm_P1.5mm_ReverseMount, B.Cu at (228.6, 128.8)
- added LED74: SK6812MINI-E, LED_SMD:LED_SK6812MINI-E_3.2x2.8mm_P1.5mm_ReverseMount, B.Cu at (247.7, 128.8)
- added LED75: SK6812MINI-E, LED_SMD:LED_SK6812MINI-E_3.2x2.8mm_P1.5mm_ReverseMount, B.Cu at (266.7, 128.8)
- added LED76: SK6812MINI-E, LED_SMD:LED_SK6812MINI-E_3.2x2.8mm_P1.5mm_ReverseMount, B.Cu at (285.8, 128.8)
- added LED77: SK6812MINI-E, LED_SMD:LED_SK6812MINI-E_3.2x2.8mm_P1.5mm_ReverseMount, B.Cu at (304.8, 128.8)
- added LED78: SK6812MINI-E, LED_SMD:LED_SK6812MINI-E_3.2x2.8mm_P1.5mm_ReverseMount, B.Cu at (347.7, 128.8)
- added LED79: SK6812MINI-E, LED_SMD:LED_SK6812MINI-E_3.2x2.8mm_P1.5mm_ReverseMount, B.Cu at (366.7, 128.8)
- added LED8: SK6812MINI-E, LED_SMD:LED_SK6812MINI-E_3.2x2.8mm_P1.5mm_ReverseMount, B.Cu at (200.0, 43.1)
- added LED80: SK6812MINI-E, LED_SMD:LED_SK6812MINI-E_3.2x2.8mm_P1.5mm_ReverseMount, B.Cu at (385.8, 128.8)
- added LED81: SK6812MINI-E, LED_SMD:LED_SK6812MINI-E_3.2x2.8mm_P1.5mm_ReverseMount, B.Cu at (40.5, 147.9)
- added LED82: SK6812MINI-E, LED_SMD:LED_SK6812MINI-E_3.2x2.8mm_P1.5mm_ReverseMount, B.Cu at (64.3, 147.9)
- added LED83: SK6812MINI-E, LED_SMD:LED_SK6812MINI-E_3.2x2.8mm_P1.5mm_ReverseMount, B.Cu at (88.1, 147.9)
- added LED84: SK6812MINI-E, LED_SMD:LED_SK6812MINI-E_3.2x2.8mm_P1.5mm_ReverseMount, B.Cu at (159.5, 147.9)
- added LED85: SK6812MINI-E, LED_SMD:LED_SK6812MINI-E_3.2x2.8mm_P1.5mm_ReverseMount, B.Cu at (231.0, 147.9)
- added LED86: SK6812MINI-E, LED_SMD:LED_SK6812MINI-E_3.2x2.8mm_P1.5mm_ReverseMount, B.Cu at (254.8, 147.9)
- added LED87: SK6812MINI-E, LED_SMD:LED_SK6812MINI-E_3.2x2.8mm_P1.5mm_ReverseMount, B.Cu at (278.6, 147.9)
- added LED88: SK6812MINI-E, LED_SMD:LED_SK6812MINI-E_3.2x2.8mm_P1.5mm_ReverseMount, B.Cu at (302.4, 147.9)
- added LED89: SK6812MINI-E, LED_SMD:LED_SK6812MINI-E_3.2x2.8mm_P1.5mm_ReverseMount, B.Cu at (347.7, 147.9)
- added LED9: SK6812MINI-E, LED_SMD:LED_SK6812MINI-E_3.2x2.8mm_P1.5mm_ReverseMount, B.Cu at (219.1, 43.1)
- added LED90: SK6812MINI-E, LED_SMD:LED_SK6812MINI-E_3.2x2.8mm_P1.5mm_ReverseMount, B.Cu at (366.7, 147.9)
- added LED91: SK6812MINI-E, LED_SMD:LED_SK6812MINI-E_3.2x2.8mm_P1.5mm_ReverseMount, B.Cu at (385.8, 147.9)
- added MX1: MX_SW_HS, PCM_marbastlib-mx:SW_MX_HS_CPG151101S11_1u, F.Cu at (38.1, 38.1)
- added MX10: MX_SW_HS, PCM_marbastlib-mx:SW_MX_HS_CPG151101S11_1u, F.Cu at (247.7, 38.1)
- added MX11: MX_SW_HS, PCM_marbastlib-mx:SW_MX_HS_CPG151101S11_1u, F.Cu at (266.7, 38.1)
- added MX12: MX_SW_HS, PCM_marbastlib-mx:SW_MX_HS_CPG151101S11_1u, F.Cu at (285.8, 38.1)
- added MX13: MX_SW_HS, PCM_marbastlib-mx:SW_MX_HS_CPG151101S11_1u, F.Cu at (304.8, 38.1)
- added MX14: MX_SW_HS, PCM_marbastlib-mx:SW_MX_HS_CPG151101S11_1u, F.Cu at (347.7, 38.1)
- added MX15: MX_SW_HS, PCM_marbastlib-mx:SW_MX_HS_CPG151101S11_1u, F.Cu at (366.7, 38.1)
- added MX16: MX_SW_HS, PCM_marbastlib-mx:SW_MX_HS_CPG151101S11_1u, F.Cu at (385.8, 38.1)
- added MX17: MX_SW_HS, PCM_marbastlib-mx:SW_MX_HS_CPG151101S11_1u, F.Cu at (38.1, 66.7)
- added MX18: MX_SW_HS, PCM_marbastlib-mx:SW_MX_HS_CPG151101S11_1u, F.Cu at (57.1, 66.7)
- added MX19: MX_SW_HS, PCM_marbastlib-mx:SW_MX_HS_CPG151101S11_1u, F.Cu at (76.2, 66.7)
- added MX2: MX_SW_HS, PCM_marbastlib-mx:SW_MX_HS_CPG151101S11_1u, F.Cu at (76.2, 38.1)
- added MX20: MX_SW_HS, PCM_marbastlib-mx:SW_MX_HS_CPG151101S11_1u, F.Cu at (95.2, 66.7)
- added MX21: MX_SW_HS, PCM_marbastlib-mx:SW_MX_HS_CPG151101S11_1u, F.Cu at (114.3, 66.7)
- added MX22: MX_SW_HS, PCM_marbastlib-mx:SW_MX_HS_CPG151101S11_1u, F.Cu at (133.3, 66.7)
- added MX23: MX_SW_HS, PCM_marbastlib-mx:SW_MX_HS_CPG151101S11_1u, F.Cu at (152.4, 66.7)
- added MX24: MX_SW_HS, PCM_marbastlib-mx:SW_MX_HS_CPG151101S11_1u, F.Cu at (171.4, 66.7)
- added MX25: MX_SW_HS, PCM_marbastlib-mx:SW_MX_HS_CPG151101S11_1u, F.Cu at (190.5, 66.7)
- added MX26: MX_SW_HS, PCM_marbastlib-mx:SW_MX_HS_CPG151101S11_1u, F.Cu at (209.6, 66.7)
- added MX27: MX_SW_HS, PCM_marbastlib-mx:SW_MX_HS_CPG151101S11_1u, F.Cu at (228.6, 66.7)
- added MX28: MX_SW_HS, PCM_marbastlib-mx:SW_MX_HS_CPG151101S11_1u, F.Cu at (247.7, 66.7)
- added MX29: MX_SW_HS, PCM_marbastlib-mx:SW_MX_HS_CPG151101S11_1u, F.Cu at (266.7, 66.7)
- added MX3: MX_SW_HS, PCM_marbastlib-mx:SW_MX_HS_CPG151101S11_1u, F.Cu at (95.2, 38.1)
- added MX30: MX_SW_HS, PCM_marbastlib-mx:SW_MX_HS_CPG151101S11_1u, F.Cu at (295.3, 66.7)
- added MX31: MX_SW_HS, PCM_marbastlib-mx:SW_MX_HS_CPG151101S11_1u, F.Cu at (347.7, 66.7)
- added MX32: MX_SW_HS, PCM_marbastlib-mx:SW_MX_HS_CPG151101S11_1u, F.Cu at (366.7, 66.7)
- added MX33: MX_SW_HS, PCM_marbastlib-mx:SW_MX_HS_CPG151101S11_1u, F.Cu at (385.8, 66.7)
- added MX34: MX_SW_HS, PCM_marbastlib-mx:SW_MX_HS_CPG151101S11_1.5u, F.Cu at (42.9, 85.7)
- added MX35: MX_SW_HS, PCM_marbastlib-mx:SW_MX_HS_CPG151101S11_1u, F.Cu at (66.7, 85.7)
- added MX36: MX_SW_HS, PCM_marbastlib-mx:SW_MX_HS_CPG151101S11_1u, F.Cu at (85.7, 85.7)
- added MX37: MX_SW_HS, PCM_marbastlib-mx:SW_MX_HS_CPG151101S11_1u, F.Cu at (104.8, 85.7)
- added MX38: MX_SW_HS, PCM_marbastlib-mx:SW_MX_HS_CPG151101S11_1u, F.Cu at (123.8, 85.7)
- added MX39: MX_SW_HS, PCM_marbastlib-mx:SW_MX_HS_CPG151101S11_1u, F.Cu at (142.9, 85.7)
- added MX4: MX_SW_HS, PCM_marbastlib-mx:SW_MX_HS_CPG151101S11_1u, F.Cu at (114.3, 38.1)
- added MX40: MX_SW_HS, PCM_marbastlib-mx:SW_MX_HS_CPG151101S11_1u, F.Cu at (161.9, 85.7)
- added MX41: MX_SW_HS, PCM_marbastlib-mx:SW_MX_HS_CPG151101S11_1u, F.Cu at (181.0, 85.7)
- added MX42: MX_SW_HS, PCM_marbastlib-mx:SW_MX_HS_CPG151101S11_1u, F.Cu at (200.0, 85.7)
- added MX43: MX_SW_HS, PCM_marbastlib-mx:SW_MX_HS_CPG151101S11_1u, F.Cu at (219.1, 85.7)
- added MX44: MX_SW_HS, PCM_marbastlib-mx:SW_MX_HS_CPG151101S11_1u, F.Cu at (238.1, 85.7)
- added MX45: MX_SW_HS, PCM_marbastlib-mx:SW_MX_HS_CPG151101S11_1u, F.Cu at (257.2, 85.7)
- added MX46: MX_SW_HS, PCM_marbastlib-mx:SW_MX_HS_CPG151101S11_1u, F.Cu at (276.2, 85.7)
- added MX47: MX_SW_HS, PCM_marbastlib-mx:SW_MX_HS_KS-2P02B01-01_1.5u, F.Cu at (300.0, 85.7)
- added MX48: MX_SW_HS, PCM_marbastlib-mx:SW_MX_HS_CPG151101S11_1u, F.Cu at (347.7, 85.7)
- added MX49: MX_SW_HS, PCM_marbastlib-mx:SW_MX_HS_CPG151101S11_1u, F.Cu at (366.7, 85.7)
- added MX5: MX_SW_HS, PCM_marbastlib-mx:SW_MX_HS_CPG151101S11_1u, F.Cu at (133.3, 38.1)
- added MX50: MX_SW_HS, PCM_marbastlib-mx:SW_MX_HS_CPG151101S11_1u, F.Cu at (385.8, 85.7)
- added MX51: MX_SW_HS, PCM_marbastlib-mx:SW_MX_HS_KS-2P02B01-01_1.75u, F.Cu at (45.2, 104.8)
- added MX52: MX_SW_HS, PCM_marbastlib-mx:SW_MX_HS_CPG151101S11_1u, F.Cu at (71.4, 104.8)
- added MX53: MX_SW_HS, PCM_marbastlib-mx:SW_MX_HS_CPG151101S11_1u, F.Cu at (90.5, 104.8)
- added MX54: MX_SW_HS, PCM_marbastlib-mx:SW_MX_HS_CPG151101S11_1u, F.Cu at (109.5, 104.8)
- added MX55: MX_SW_HS, PCM_marbastlib-mx:SW_MX_HS_CPG151101S11_1u, F.Cu at (128.6, 104.8)
- added MX56: MX_SW_HS, PCM_marbastlib-mx:SW_MX_HS_CPG151101S11_1u, F.Cu at (147.6, 104.8)
- added MX57: MX_SW_HS, PCM_marbastlib-mx:SW_MX_HS_CPG151101S11_1u, F.Cu at (166.7, 104.8)
- added MX58: MX_SW_HS, PCM_marbastlib-mx:SW_MX_HS_CPG151101S11_1u, F.Cu at (185.7, 104.8)
- added MX59: MX_SW_HS, PCM_marbastlib-mx:SW_MX_HS_CPG151101S11_1u, F.Cu at (204.8, 104.8)
- added MX6: MX_SW_HS, PCM_marbastlib-mx:SW_MX_HS_CPG151101S11_1u, F.Cu at (161.9, 38.1)
- added MX60: MX_SW_HS, PCM_marbastlib-mx:SW_MX_HS_CPG151101S11_1u, F.Cu at (223.8, 104.8)
- added MX61: MX_SW_HS, PCM_marbastlib-mx:SW_MX_HS_CPG151101S11_1u, F.Cu at (242.9, 104.8)
- added MX62: MX_SW_HS, PCM_marbastlib-mx:SW_MX_HS_CPG151101S11_1u, F.Cu at (261.9, 104.8)
- added MX63: MX_SW_HS, PCM_marbastlib-mx:SW_MX_HS_CPG151101S11_1u, F.Cu at (292.9, 104.8)
- added MX64: MX_SW_HS, PCM_marbastlib-mx:SW_MX_HS_CPG151101S11_1u, F.Cu at (47.6, 123.8)
- added MX65: MX_SW_HS, PCM_marbastlib-mx:SW_MX_HS_CPG151101S11_1u, F.Cu at (76.2, 123.8)
- added MX66: MX_SW_HS, PCM_marbastlib-mx:SW_MX_HS_CPG151101S11_1u, F.Cu at (95.2, 123.8)
- added MX67: MX_SW_HS, PCM_marbastlib-mx:SW_MX_HS_CPG151101S11_1u, F.Cu at (114.3, 123.8)
- added MX68: MX_SW_HS, PCM_marbastlib-mx:SW_MX_HS_CPG151101S11_1u, F.Cu at (133.3, 123.8)
- added MX69: MX_SW_HS, PCM_marbastlib-mx:SW_MX_HS_CPG151101S11_1u, F.Cu at (152.4, 123.8)
- added MX7: MX_SW_HS, PCM_marbastlib-mx:SW_MX_HS_CPG151101S11_1u, F.Cu at (181.0, 38.1)
- added MX70: MX_SW_HS, PCM_marbastlib-mx:SW_MX_HS_CPG151101S11_1u, F.Cu at (171.4, 123.8)
- added MX71: MX_SW_HS, PCM_marbastlib-mx:SW_MX_HS_CPG151101S11_1u, F.Cu at (190.5, 123.8)
- added MX72: MX_SW_HS, PCM_marbastlib-mx:SW_MX_HS_CPG151101S11_1u, F.Cu at (209.6, 123.8)
- added MX73: MX_SW_HS, PCM_marbastlib-mx:SW_MX_HS_CPG151101S11_1u, F.Cu at (228.6, 123.8)
- added MX74: MX_SW_HS, PCM_marbastlib-mx:SW_MX_HS_CPG151101S11_1u, F.Cu at (247.7, 123.8)
- added MX75: MX_SW_HS, PCM_marbastlib-mx:SW_MX_HS_CPG151101S11_1u, F.Cu at (266.7, 123.8)
- added MX76: MX_SW_HS, PCM_marbastlib-mx:SW_MX_HS_CPG151101S11_1u, F.Cu at (285.8, 123.8)
- added MX77: MX_SW_HS, PCM_marbastlib-mx:SW_MX_HS_CPG151101S11_1u, F.Cu at (304.8, 123.8)
- added MX78: MX_SW_HS, PCM_marbastlib-mx:SW_MX_HS_CPG151101S11_1u, F.Cu at (347.7, 123.8)
- added MX79: MX_SW_HS, PCM_marbastlib-mx:SW_MX_HS_CPG151101S11_1u, F.Cu at (366.7, 123.8)
- added MX8: MX_SW_HS, PCM_marbastlib-mx:SW_MX_HS_CPG151101S11_1u, F.Cu at (200.0, 38.1)
- added MX80: MX_SW_HS, PCM_marbastlib-mx:SW_MX_HS_CPG151101S11_1u, F.Cu at (385.8, 123.8)
- added MX81: MX_SW_HS, PCM_marbastlib-mx:SW_MX_HS_KS-2P02B01-01_1.25u, F.Cu at (40.5, 142.9)
- added MX82: MX_SW_HS, PCM_marbastlib-mx:SW_MX_HS_KS-2P02B01-01_1.25u, F.Cu at (64.3, 142.9)
- added MX83: MX_SW_HS, PCM_marbastlib-mx:SW_MX_HS_KS-2P02B01-01_1.25u, F.Cu at (88.1, 142.9)
- added MX84: MX_SW_HS, PCM_marbastlib-mx:SW_MX_HS_CPG151101S11_1.25u, F.Cu at (159.5, 142.9)
- added MX85: MX_SW_HS, PCM_marbastlib-mx:SW_MX_HS_KS-2P02B01-01_1.25u, F.Cu at (231.0, 142.9)
- added MX86: MX_SW_HS, PCM_marbastlib-mx:SW_MX_HS_KS-2P02B01-01_1.25u, F.Cu at (254.8, 142.9)
- added MX87: MX_SW_HS, PCM_marbastlib-mx:SW_MX_HS_KS-2P02B01-01_1.25u, F.Cu at (278.6, 142.9)
- added MX88: MX_SW_HS, PCM_marbastlib-mx:SW_MX_HS_KS-2P02B01-01_1.25u, F.Cu at (302.4, 142.9)
- added MX89: MX_SW_HS, PCM_marbastlib-mx:SW_MX_HS_CPG151101S11_1u, F.Cu at (347.7, 142.9)
- added MX9: MX_SW_HS, PCM_marbastlib-mx:SW_MX_HS_CPG151101S11_1u, F.Cu at (219.1, 38.1)
- added MX90: MX_SW_HS, PCM_marbastlib-mx:SW_MX_HS_CPG151101S11_1u, F.Cu at (366.7, 142.9)
- added MX91: MX_SW_HS, PCM_marbastlib-mx:SW_MX_HS_CPG151101S11_1u, F.Cu at (385.8, 142.9)
- added R1: 470, Resistor_THT:R_Axial_DIN0207_L6.3mm_D2.5mm_P7.62mm_Horizontal, F.Cu at (18.6, 181.8)
- added S1: MX_stab, PCM_marbastlib-mx:STAB_MX_P_6.25u, F.Cu at (119.8, 266.7)
- added S2: MX_stab, PCM_marbastlib-mx:STAB_MX_2u, F.Cu at (81.8, 206.4)
- added S3: MX_stab, PCM_marbastlib-mx:STAB_MX_2u, F.Cu at (81.8, 226.7)
- added S4: MX_stab, PCM_marbastlib-mx:STAB_MX_2.25u, F.Cu at (81.8, 247.0)
- moved A1 344.3 mm to (32.4, 223.5)
- moved D55 0.91 mm to (136.9, 106.9)
- moved D60 0.91 mm to (232.1, 106.9)
- moved D69 0.91 mm to (160.7, 125.9)
- moved D74 0.91 mm to (255.9, 125.9)
- moved D75 0.91 mm to (275.0, 125.9)
- moved D78 0.91 mm to (356.0, 125.9)
- moved D79 0.91 mm to (375.0, 125.9)
- moved D80 0.91 mm to (394.1, 125.9)
- moved D86 0.91 mm to (263.1, 145.0)
- moved D87 0.91 mm to (286.9, 145.0)
- moved D88 0.91 mm to (310.7, 145.0)
- moved D89 0.91 mm to (356.0, 145.0)
- moved D90 0.91 mm to (375.0, 145.0)
- moved D91 0.91 mm to (394.1, 145.0)
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Connections:
- A1 pad 33: GND -> unconnected-(A1-AGND-Pad33)
- A1 pad 40: unconnected-(A1-VBUS-Pad40) -> +5V
Routing:
- net /Row0: track 347.9 -> 0.00 mm
- net /Row1: track 347.7 -> 0.00 mm
- net /Row5: track 345.3 -> 0.00 mm
- net /Row2: track 342.9 -> 0.00 mm
- net /Row4: track 338.1 -> 0.00 mm
- net /Row3: track 247.6 -> 0.00 mm
- net /Col11: track 125.5 -> 0.00 mm
- net /Col10: track 123.5 -> 0.00 mm
- net /Col13: track 120.5 -> 0.00 mm
- net /Col9: track 117.6 -> 0.00 mm
- net /Col2: track 115.6 -> 0.00 mm
- net /Col5: track 115.6 -> 0.00 mm
- net /Col0: track 111.7 -> 0.00 mm
- net /Col16: track 104.8 -> 0.00 mm
- net /Col15: track 104.8 -> 0.00 mm
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- removed copper zone on B.Cu, net GND
Other:
- board outline added: 3.6 x 3.2 mm

Commit message: Started wiring, and fixed pcb's rgbs data line going across the whole board
Parts:
- S1: footprint PCM_marbastlib-mx:STAB_MX_P_6.25u -> PCM_marbastlib-mx:STAB_MX_6.25u
- moved A1 344.4 mm to (317.4, 30.1)
- moved S3 266.8 mm to (295.3, 66.7)
- moved S4 254.6 mm to (292.9, 104.8)
- moved H1 237.5 mm to (19.1, 157.2)
- moved H2 237.5 mm to (23.8, 157.2)
- moved H3 237.5 mm to (28.6, 157.2)
- moved H4 237.5 mm to (33.3, 157.2)
- moved S1 130.0 mm to (159.5, 142.9)
- moved S2 89.3 mm to (47.6, 123.8)
- moved R1 15.3 mm to (21.0, 166.7)
Routing:
- net /Row5: track 0.00 -> 347.4 mm
- net /Row2: track 0.00 -> 346.2 mm
- net /Row4: track 0.00 -> 341.5 mm
- net /Row0: track 0.00 -> 307.8 mm
- net /Row1: track 0.00 -> 298.5 mm
- net /Row3: track 0.00 -> 250.2 mm
- net /Col11: track 0.00 -> 125.5 mm
- net /Col10: track 0.00 -> 123.5 mm
- net /Col13: track 0.00 -> 121.7 mm
- net /Col9: track 0.00 -> 117.6 mm
- net /Col5: track 0.00 -> 115.6 mm
- net /Col2: track 0.00 -> 114.2 mm
- net /Col0: track 0.00 -> 113.8 mm
- net /Col16: track 0.00 -> 104.8 mm
- net /Col15: track 0.00 -> 104.8 mm
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