File: keyboard-full/keyboard-full.kicad_pcb (KiCad board)
At the start: 2 copper layers, 3.6 x 3.2 mm, 374 parts

Commit message: Finished up wiring
Parts:
- moved H2 335.4 mm to (392.9, 111.1)
- moved S3 282.1 mm to (295.3, 66.7)
- moved S4 272.7 mm to (292.9, 104.8)
- moved H3 236.0 mm to (234.1, 35.7)
- moved R1 210.4 mm to (29.4, 35.9), turned to -90 degrees
- moved H4 148.0 mm to (200.0, 141.3)
- moved H1 145.9 mm to (32.5, 51.6)
- moved S1 124.6 mm to (159.5, 142.9)
- moved S2 44.2 mm to (47.6, 123.8)
- moved C17 0.22 mm to (38.3, 74.8)
Connections:
- A1 pad 1: unconnected-(A1-GPIO0-Pad1) -> /LED
- A1 pad 10: unconnected-(A1-GPIO7-Pad10) -> /Col4
- A1 pad 11: unconnected-(A1-GPIO8-Pad11) -> /Col5
- A1 pad 12: unconnected-(A1-GPIO9-Pad12) -> /Col6
- A1 pad 14: unconnected-(A1-GPIO10-Pad14) -> /Col7
- A1 pad 15: unconnected-(A1-GPIO11-Pad15) -> /Col8
- A1 pad 16: unconnected-(A1-GPIO12-Pad16) -> /Col9
- A1 pad 17: unconnected-(A1-GPIO13-Pad17) -> /Col10
- A1 pad 19: unconnected-(A1-GPIO14-Pad19) -> /Col11
- A1 pad 2: unconnected-(A1-GPIO1-Pad2) -> /Col13
- A1 pad 20: unconnected-(A1-GPIO15-Pad20) -> /Col12
- A1 pad 21: unconnected-(A1-GPIO16-Pad21) -> /Row5
- A1 pad 22: /Row5 -> /Row4
- A1 pad 24: /Row4 -> /Row3
- A1 pad 25: /Row3 -> /Row2
- A1 pad 26: /Row2 -> /Row1
- A1 pad 27: /Row1 -> unconnected-(A1-GPIO21-Pad27)
- A1 pad 29: /Row0 -> unconnected-(A1-GPIO22-Pad29)
- A1 pad 31: /Col14 -> /Col16
- A1 pad 34: /Col16 -> /Col14
- A1 pad 4: unconnected-(A1-GPIO2-Pad4) -> /Row0
- A1 pad 5: unconnected-(A1-GPIO3-Pad5) -> /Col0
- A1 pad 6: unconnected-(A1-GPIO4-Pad6) -> /Col1
- A1 pad 7: unconnected-(A1-GPIO5-Pad7) -> /Col2
- A1 pad 9: unconnected-(A1-GPIO6-Pad9) -> /Col3
Routing:
- net +5V: track 445.6 -> 2874.1 mm, vias 80 -> 89
- net /Col0: track 0.00 -> 401.3 mm, vias 0 -> 1
- net /Col1: track 0.00 -> 360.9 mm, vias 0 -> 1
- net /Col2: track 0.00 -> 358.1 mm, vias 0 -> 1
- net /Row1: track 38.5 -> 353.7 mm
- net /Col3: track 0.00 -> 313.3 mm, vias 0 -> 1
- net /Col5: track 0.00 -> 300.2 mm, vias 0 -> 1
- net /Col4: track 0.00 -> 295.4 mm, vias 0 -> 1
- net /LED: track 0.00 -> 292.4 mm
- net /Col6: track 0.00 -> 253.9 mm, vias 0 -> 1
- net /Col7: track 0.00 -> 240.4 mm, vias 0 -> 1
- net /Col9: track 0.00 -> 228.4 mm, vias 0 -> 1
- net /Col8: track 0.00 -> 226.0 mm, vias 0 -> 1
- net /Col10: track 0.00 -> 208.3 mm, vias 0 -> 1
- net /Col11: track 0.00 -> 206.4 mm, vias 0 -> 1
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
Commit message: Finished pcb design
Routing:
- net +5V: track 2874.1 -> 2817.5 mm
- net /Row0: track 354.9 -> 362.5 mm, vias 0 -> 16
- net /Row2: track 366.9 -> 374.1 mm, vias 1 -> 18
- net /Row4: track 392.6 -> 396.8 mm, vias 1 -> 12
- net Net-(LED30-DIN): track 59.9 -> 61.8 mm
- net /Col12: track 168.1 -> 168.8 mm
- net GND: vias 0 -> 87
- added copper zone on B.Cu, net GND
- added copper zone on F.Cu, net GND
Other:
- board size 3.6 x 3.2 mm -> 369.8 x 125.4 mm
