File: keyboard-full/keyboard-full.kicad_pcb (KiCad board)
At the start: 2 copper layers, 369.8 x 125.4 mm, 374 parts

Commit message: redid the keyboard pcb design
Parts:
- removed the H3 at (234.1, 35.7)
- added H3: MountingHole, MountingHole:MountingHole_2.1mm, F.Cu at (190.0, 95.0)
- added H3: MountingHole, MountingHole:MountingHole_2.1mm, F.Cu at (54.8, 136.5)
- MX1, MX10, MX11, MX12, MX13, MX14, MX15, MX16, MX17, MX18, MX19, MX2, MX20, MX21, MX22, MX23, MX24, MX25, MX26, MX27, MX28, MX29, MX3, MX30, MX31, MX32, MX33, MX34, MX35, MX36, MX37, MX38, MX39, MX4, MX40, MX41, MX42, MX43, MX44, MX45, MX46, MX48, MX49, MX5, MX50, MX52, MX53, MX54, MX55, MX56, MX57, MX58, MX59, MX6, MX60, MX61, MX62, MX63, MX64, MX65, MX66, MX67, MX68, MX69, MX7, MX70, MX71, MX72, MX73, MX74, MX75, MX76, MX77, MX78, MX79, MX8, MX80, MX84, MX89, MX9, MX90, MX91: moved to B.Cu
- MX47: footprint PCM_marbastlib-mx:SW_MX_HS_KS-2P02B01-01_1.5u -> PCM_marbastlib-mx:SW_MX_HS_CPG151101S11_1.5u; moved to B.Cu
- MX51: footprint PCM_marbastlib-mx:SW_MX_HS_KS-2P02B01-01_1.75u -> PCM_marbastlib-mx:SW_MX_HS_CPG151101S11_1.75u; moved to B.Cu
- MX81, MX82, MX83, MX85, MX86, MX87, MX88: footprint PCM_marbastlib-mx:SW_MX_HS_KS-2P02B01-01_1.25u -> PCM_marbastlib-mx:SW_MX_HS_CPG151101S11_1.25u; moved to B.Cu
- R1: value 470 -> R470
- moved R1 284.1 mm to (313.3, 46.3)
- moved H4 136.1 mm to (335.7, 150.8)
- moved H2 58.7 mm to (392.1, 52.4)
- moved H1 7.19 mm to (39.7, 52.4)
- moved C33 5.55 mm to (380.8, 72.4), turned to -90 degrees
- moved C12 5.49 mm to (280.8, 43.8), turned to -90 degrees
- moved C11 5.49 mm to (261.7, 43.8), turned to -90 degrees
- moved C46 5.48 mm to (271.3, 91.4), turned to -90 degrees
- moved C47 5.48 mm to (295.1, 91.4), turned to -90 degrees
- moved C37 5.48 mm to (99.8, 91.4), turned to -90 degrees
- moved C39 5.48 mm to (137.9, 91.4), turned to -90 degrees
- moved C40 5.48 mm to (157.0, 91.4), turned to -90 degrees
- moved C42 5.48 mm to (195.1, 91.4), turned to -90 degrees
- moved C44 5.48 mm to (233.2, 91.4), turned to -90 degrees
- moved C45 5.48 mm to (252.2, 91.4), turned to -90 degrees
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Connections:
- A1 pad 1: /LED -> /Row0
- A1 pad 10: /Col4 -> /Col6
- A1 pad 11: /Col5 -> /Col7
- A1 pad 12: /Col6 -> /LED
- A1 pad 14: /Col7 -> /Col8
- A1 pad 15: /Col8 -> /Col9
- A1 pad 16: /Col9 -> /Col10
- A1 pad 17: /Col10 -> /Col11
- A1 pad 19: /Col11 -> /Col12
- A1 pad 2: /Col13 -> /Col0
- A1 pad 20: /Col12 -> /Col13
- A1 pad 4: /Row0 -> /Col1
- A1 pad 5: /Col0 -> /Col2
- A1 pad 6: /Col1 -> /Col3
- A1 pad 7: /Col2 -> /Col4
- A1 pad 9: /Col3 -> /Col5
- C25 pad 2: GND -> unconnected-(C25-Pad2)
- LED11 pad 2: Net-(LED10-DOUT) -> Net-(LED11-DIN)
- LED11 pad 4: Net-(LED11-DOUT) -> Net-(LED10-DIN)
- LED12 pad 2: Net-(LED11-DOUT) -> Net-(LED12-DIN)
- LED12 pad 4: Net-(LED12-DOUT) -> Net-(LED11-DIN)
- LED13 pad 2: Net-(LED12-DOUT) -> Net-(LED13-DIN)
- LED13 pad 4: Net-(LED13-DOUT) -> Net-(LED12-DIN)
- LED14 pad 2: Net-(LED13-DOUT) -> Net-(LED14-DIN)
- LED16 pad 4: Net-(LED16-DOUT) -> unconnected-(LED16-DOUT-Pad4)
- LED17 pad 2: Net-(LED17-DIN) -> Net-(LED1-DOUT)
- LED18 pad 2: Net-(LED18-DIN) -> Net-(LED17-DOUT)
- LED18 pad 4: Net-(LED17-DIN) -> Net-(LED18-DOUT)
- LED19 pad 2: Net-(LED19-DIN) -> Net-(LED18-DOUT)
- LED19 pad 4: Net-(LED18-DIN) -> Net-(LED19-DOUT)
- LED2 pad 2: Net-(LED1-DOUT) -> Net-(LED2-DIN)
- LED2 pad 4: Net-(LED2-DOUT) -> Net-(LED1-DIN)
- LED20 pad 2: Net-(LED20-DIN) -> Net-(LED19-DOUT)
- LED20 pad 4: Net-(LED19-DIN) -> Net-(LED20-DOUT)
- LED21 pad 2: Net-(LED21-DIN) -> Net-(LED20-DOUT)
- LED21 pad 4: Net-(LED20-DIN) -> Net-(LED21-DOUT)
- LED22 pad 2: Net-(LED22-DIN) -> Net-(LED21-DOUT)
- LED22 pad 4: Net-(LED21-DIN) -> Net-(LED22-DOUT)
- LED23 pad 2: Net-(LED23-DIN) -> Net-(LED22-DOUT)
- LED23 pad 4: Net-(LED22-DIN) -> Net-(LED23-DOUT)
- LED24 pad 2: Net-(LED24-DIN) -> Net-(LED23-DOUT)
- LED24 pad 4: Net-(LED23-DIN) -> Net-(LED24-DOUT)
- LED25 pad 2: Net-(LED25-DIN) -> Net-(LED24-DOUT)
- LED25 pad 4: Net-(LED24-DIN) -> Net-(LED25-DOUT)
- LED26 pad 2: Net-(LED26-DIN) -> Net-(LED25-DOUT)
- LED26 pad 4: Net-(LED25-DIN) -> Net-(LED26-DOUT)
- LED27 pad 2: Net-(LED27-DIN) -> Net-(LED26-DOUT)
- LED27 pad 4: Net-(LED26-DIN) -> Net-(LED27-DOUT)
- LED28 pad 2: Net-(LED28-DIN) -> Net-(LED27-DOUT)
- LED28 pad 4: Net-(LED27-DIN) -> Net-(LED28-DOUT)
- LED29 pad 2: Net-(LED29-DIN) -> Net-(LED28-DOUT)
- LED29 pad 4: Net-(LED28-DIN) -> Net-(LED29-DOUT)
- LED3 pad 2: Net-(LED2-DOUT) -> Net-(LED3-DIN)
- LED3 pad 4: Net-(LED3-DOUT) -> Net-(LED2-DIN)
- LED30 pad 2: Net-(LED30-DIN) -> Net-(LED29-DOUT)
- LED30 pad 4: Net-(LED29-DIN) -> Net-(LED30-DOUT)
- LED31 pad 4: Net-(LED30-DIN) -> Net-(LED14-DIN)
- LED33 pad 2: Net-(LED16-DOUT) -> Net-(LED33-DIN)
- LED34 pad 2: Net-(LED17-DOUT) -> Net-(LED34-DIN)
- LED35 pad 2: Net-(LED34-DOUT) -> Net-(LED35-DIN)
- LED35 pad 4: Net-(LED35-DOUT) -> Net-(LED34-DIN)
- LED36 pad 2: Net-(LED35-DOUT) -> Net-(LED36-DIN)
- LED36 pad 4: Net-(LED36-DOUT) -> Net-(LED35-DIN)
- LED37 pad 2: Net-(LED36-DOUT) -> Net-(LED37-DIN)
- LED37 pad 4: Net-(LED37-DOUT) -> Net-(LED36-DIN)
- LED38 pad 2: Net-(LED37-DOUT) -> Net-(LED38-DIN)
- LED38 pad 4: Net-(LED38-DOUT) -> Net-(LED37-DIN)
- LED39 pad 2: Net-(LED38-DOUT) -> Net-(LED39-DIN)
- LED39 pad 4: Net-(LED39-DOUT) -> Net-(LED38-DIN)
- LED4 pad 2: Net-(LED3-DOUT) -> Net-(LED4-DIN)
- LED4 pad 4: Net-(LED4-DOUT) -> Net-(LED3-DIN)
- LED40 pad 2: Net-(LED39-DOUT) -> Net-(LED40-DIN)
- LED40 pad 4: Net-(LED40-DOUT) -> Net-(LED39-DIN)
- LED41 pad 2: Net-(LED40-DOUT) -> Net-(LED41-DIN)
- LED41 pad 4: Net-(LED41-DOUT) -> Net-(LED40-DIN)
- LED42 pad 2: Net-(LED41-DOUT) -> Net-(LED42-DIN)
- LED42 pad 4: Net-(LED42-DOUT) -> Net-(LED41-DIN)
- LED43 pad 2: Net-(LED42-DOUT) -> Net-(LED43-DIN)
- LED43 pad 4: Net-(LED43-DOUT) -> Net-(LED42-DIN)
- LED44 pad 2: Net-(LED43-DOUT) -> Net-(LED44-DIN)
- LED44 pad 4: Net-(LED44-DOUT) -> Net-(LED43-DIN)
- LED45 pad 2: Net-(LED44-DOUT) -> Net-(LED45-DIN)
- LED45 pad 4: Net-(LED45-DOUT) -> Net-(LED44-DIN)
- LED46 pad 2: Net-(LED45-DOUT) -> Net-(LED46-DIN)
- LED46 pad 4: Net-(LED46-DOUT) -> Net-(LED45-DIN)
- LED47 pad 2: Net-(LED46-DOUT) -> Net-(LED30-DOUT)
- LED47 pad 4: Net-(LED47-DOUT) -> Net-(LED46-DIN)
- LED48 pad 2: Net-(LED47-DOUT) -> Net-(LED48-DIN)
- LED5 pad 2: Net-(LED4-DOUT) -> Net-(LED5-DIN)
- LED5 pad 4: Net-(LED5-DOUT) -> Net-(LED4-DIN)
- LED50 pad 4: Net-(LED50-DOUT) -> Net-(LED33-DIN)
- LED51 pad 2: Net-(LED51-DIN) -> Net-(LED34-DOUT)
- LED52 pad 2: Net-(LED52-DIN) -> Net-(LED51-DOUT)
- LED52 pad 4: Net-(LED51-DIN) -> Net-(LED52-DOUT)
- LED53 pad 2: Net-(LED53-DIN) -> Net-(LED52-DOUT)
- LED53 pad 4: Net-(LED52-DIN) -> Net-(LED53-DOUT)
- LED54 pad 2: Net-(LED54-DIN) -> Net-(LED53-DOUT)
- LED54 pad 4: Net-(LED53-DIN) -> Net-(LED54-DOUT)
- LED55 pad 2: Net-(LED55-DIN) -> Net-(LED54-DOUT)
- LED55 pad 4: Net-(LED54-DIN) -> Net-(LED55-DOUT)
- LED56 pad 2: Net-(LED56-DIN) -> Net-(LED55-DOUT)
- LED56 pad 4: Net-(LED55-DIN) -> Net-(LED56-DOUT)
- LED57 pad 2: Net-(LED57-DIN) -> Net-(LED56-DOUT)
- LED57 pad 4: Net-(LED56-DIN) -> Net-(LED57-DOUT)
- LED58 pad 2: Net-(LED58-DIN) -> Net-(LED57-DOUT)
- LED58 pad 4: Net-(LED57-DIN) -> Net-(LED58-DOUT)
- LED59 pad 2: Net-(LED59-DIN) -> Net-(LED58-DOUT)
- LED59 pad 4: Net-(LED58-DIN) -> Net-(LED59-DOUT)
- LED6 pad 2: Net-(LED5-DOUT) -> Net-(LED6-DIN)
- LED6 pad 4: Net-(LED6-DOUT) -> Net-(LED5-DIN)
- LED60 pad 2: Net-(LED60-DIN) -> Net-(LED59-DOUT)
- LED60 pad 4: Net-(LED59-DIN) -> Net-(LED60-DOUT)
- LED61 pad 2: Net-(LED61-DIN) -> Net-(LED60-DOUT)
- LED61 pad 4: Net-(LED60-DIN) -> Net-(LED61-DOUT)
- LED62 pad 2: Net-(LED62-DIN) -> Net-(LED61-DOUT)
- LED62 pad 4: Net-(LED61-DIN) -> Net-(LED62-DOUT)
- LED63 pad 2: Net-(LED50-DOUT) -> Net-(LED62-DOUT)
- LED63 pad 4: Net-(LED62-DIN) -> Net-(LED63-DOUT)
- LED64 pad 2: Net-(LED51-DOUT) -> Net-(LED64-DIN)
- LED65 pad 2: Net-(LED64-DOUT) -> Net-(LED65-DIN)
- LED65 pad 4: Net-(LED65-DOUT) -> Net-(LED64-DIN)
- LED66 pad 2: Net-(LED65-DOUT) -> Net-(LED66-DIN)
- LED66 pad 4: Net-(LED66-DOUT) -> Net-(LED65-DIN)
- LED67 pad 2: Net-(LED66-DOUT) -> Net-(LED67-DIN)
- LED67 pad 4: Net-(LED67-DOUT) -> Net-(LED66-DIN)
- LED68 pad 2: Net-(LED67-DOUT) -> Net-(LED68-DIN)
- LED68 pad 4: Net-(LED68-DOUT) -> Net-(LED67-DIN)
- LED69 pad 2: Net-(LED68-DOUT) -> Net-(LED69-DIN)
- LED69 pad 4: Net-(LED69-DOUT) -> Net-(LED68-DIN)
- LED7 pad 2: Net-(LED6-DOUT) -> Net-(LED7-DIN)
- LED7 pad 4: Net-(LED7-DOUT) -> Net-(LED6-DIN)
- LED70 pad 2: Net-(LED69-DOUT) -> Net-(LED70-DIN)
- LED70 pad 4: Net-(LED70-DOUT) -> Net-(LED69-DIN)
- LED71 pad 2: Net-(LED70-DOUT) -> Net-(LED71-DIN)
- LED71 pad 4: Net-(LED71-DOUT) -> Net-(LED70-DIN)
- LED72 pad 2: Net-(LED71-DOUT) -> Net-(LED72-DIN)
- LED72 pad 4: Net-(LED72-DOUT) -> Net-(LED71-DIN)
- LED73 pad 2: Net-(LED72-DOUT) -> Net-(LED73-DIN)
- LED73 pad 4: Net-(LED73-DOUT) -> Net-(LED72-DIN)
- LED74 pad 2: Net-(LED73-DOUT) -> Net-(LED74-DIN)
- LED74 pad 4: Net-(LED74-DOUT) -> Net-(LED73-DIN)
- LED75 pad 2: Net-(LED74-DOUT) -> Net-(LED75-DIN)
- LED75 pad 4: Net-(LED75-DOUT) -> Net-(LED74-DIN)
- LED76 pad 2: Net-(LED75-DOUT) -> Net-(LED76-DIN)
- LED76 pad 4: Net-(LED76-DOUT) -> Net-(LED75-DIN)
- LED77 pad 2: Net-(LED76-DOUT) -> Net-(LED63-DOUT)
- LED77 pad 4: Net-(LED77-DOUT) -> Net-(LED76-DIN)
- LED78 pad 2: Net-(LED77-DOUT) -> Net-(LED78-DIN)
- LED78 pad 4: Net-(LED78-DOUT) -> Net-(LED48-DIN)
- LED79 pad 2: Net-(LED78-DOUT) -> Net-(LED79-DIN)
- LED79 pad 4: Net-(LED79-DOUT) -> Net-(LED78-DIN)
- LED8 pad 2: Net-(LED7-DOUT) -> Net-(LED8-DIN)
- LED8 pad 4: Net-(LED8-DOUT) -> Net-(LED7-DIN)
- LED80 pad 2: Net-(LED79-DOUT) -> Net-(LED80-DIN)
- LED80 pad 4: Net-(LED80-DOUT) -> Net-(LED79-DIN)
- LED81 pad 2: Net-(LED81-DIN) -> Net-(LED64-DOUT)
- LED81 pad 4: unconnected-(LED81-DOUT-Pad4) -> Net-(LED81-DOUT)
- LED82 pad 2: Net-(LED82-DIN) -> Net-(LED81-DOUT)
- LED82 pad 4: Net-(LED81-DIN) -> Net-(LED82-DOUT)
- LED83 pad 2: Net-(LED83-DIN) -> Net-(LED82-DOUT)
- LED83 pad 4: Net-(LED82-DIN) -> Net-(LED83-DOUT)
- LED84 pad 2: Net-(LED84-DIN) -> Net-(LED83-DOUT)
- LED84 pad 4: Net-(LED83-DIN) -> Net-(LED84-DOUT)
- LED85 pad 2: Net-(LED85-DIN) -> Net-(LED84-DOUT)
- LED85 pad 4: Net-(LED84-DIN) -> Net-(LED85-DOUT)
- LED86 pad 2: Net-(LED86-DIN) -> Net-(LED85-DOUT)
- LED86 pad 4: Net-(LED85-DIN) -> Net-(LED86-DOUT)
- LED87 pad 2: Net-(LED87-DIN) -> Net-(LED86-DOUT)
- LED87 pad 4: Net-(LED86-DIN) -> Net-(LED87-DOUT)
- LED88 pad 2: Net-(LED88-DIN) -> Net-(LED87-DOUT)
- LED88 pad 4: Net-(LED87-DIN) -> Net-(LED88-DOUT)
- LED89 pad 2: Net-(LED89-DIN) -> Net-(LED88-DOUT)
- LED89 pad 4: Net-(LED88-DIN) -> Net-(LED89-DOUT)
- LED9 pad 2: Net-(LED8-DOUT) -> Net-(LED10-DOUT)
- LED9 pad 4: Net-(LED10-DIN) -> Net-(LED8-DIN)
- LED90 pad 2: Net-(LED90-DIN) -> Net-(LED89-DOUT)
- LED90 pad 4: Net-(LED89-DIN) -> Net-(LED90-DOUT)
- LED91 pad 2: Net-(LED80-DOUT) -> Net-(LED90-DOUT)
- LED91 pad 4: Net-(LED90-DIN) -> Net-(LED80-DIN)
- R1 pad 1: /LED -> Net-(LED13-DIN)
- R1 pad 2: Net-(LED1-DIN) -> /LED
Routing:
- net +5V: track 2817.5 -> 3211.1 mm, vias 89 -> 90
- net /LED: track 292.4 -> 5.90 mm
- net Net-(LED50-DOUT): track 104.2 -> 0.00 mm
- net Net-(LED83-DIN): track 66.8 -> 0.00 mm
- net Net-(LED84-DIN): track 66.8 -> 0.00 mm
- net Net-(LED83-DOUT): track 0.00 -> 66.6 mm
- net Net-(LED84-DOUT): track 0.00 -> 66.6 mm
- net Net-(LED30-DIN): track 61.8 -> 0.00 mm
- net Net-(LED48-DIN): track 0.00 -> 50.2 mm, vias 0 -> 2
- net Net-(LED47-DOUT): track 42.8 -> 0.00 mm
- net Net-(LED13-DOUT): track 40.9 -> 0.00 mm
- net Net-(LED88-DOUT): track 0.00 -> 40.4 mm
- net Net-(LED88-DIN): track 40.4 -> 0.00 mm
- net Net-(LED77-DOUT): track 38.0 -> 0.00 mm
- net Net-(LED16-DOUT): track 37.2 -> 0.00 mm
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Other:
- board size 369.8 x 125.4 mm -> 368.3 x 125.4 mm
