File: keyboard-full/keyboard-full.kicad_sch (KiCad schematic)
At the start: 374 parts

Commit message: Finished up wiring
Connections:
- net Col0: now also A1.5 (GPIO3)
- net Col1: now also A1.6 (GPIO4)
- net Col10: now also A1.17 (GPIO13)
- net Col11: now also A1.19 (GPIO14)
- net Col12: now also A1.20 (GPIO15)
- net Col13: now also A1.2 (GPIO1)
- net Col14: now also A1.34 (GPIO28_ADC2); no longer A1.31 (GPIO26_ADC0)
- net Col16: now also A1.31 (GPIO26_ADC0); no longer A1.34 (GPIO28_ADC2)
- net Col2: now also A1.7 (GPIO5)
- net Col3: now also A1.9 (GPIO6)
- net Col4: now also A1.10 (GPIO7)
- net Col5: now also A1.11 (GPIO8)
- net Col6: now also A1.12 (GPIO9)
- net Col7: now also A1.14 (GPIO10)
- net Col8: now also A1.15 (GPIO11)
- net Col9: now also A1.16 (GPIO12)
- net LED: now also A1.1 (GPIO0)
- net Row0: now also A1.4 (GPIO2); no longer A1.29 (GPIO22)
- net Row1: now also A1.26 (GPIO20); no longer A1.27 (GPIO21)
- net Row2: now also A1.25 (GPIO19); no longer A1.26 (GPIO20)
- net Row3: now also A1.24 (GPIO18); no longer A1.25 (GPIO19)
- net Row4: now also A1.22 (GPIO17); no longer A1.24 (GPIO18)
- net Row5: now also A1.21 (GPIO16); no longer A1.22 (GPIO17)
