File: keyboard-full/_restore_backup_2026-09-18T17-51-47-894/keyboard-full.kicad_pcb (KiCad board)
At the start: 2 copper layers, 3.6 x 3.2 mm, 374 parts

Commit message: Done some wiring
Parts:
- moved C33 0.15 mm to (385.8, 74.7), turned to 180 degrees
- turned C17 to 180 degrees
- turned C18 to 180 degrees
- turned C19 to 180 degrees
- turned C20 to 180 degrees
- turned C21 to 180 degrees
- turned C22 to 180 degrees
- turned C23 to 180 degrees
- turned C24 to 180 degrees
- turned C25 to 180 degrees
- turned C26 to 180 degrees
- turned C27 to 180 degrees
- turned C28 to 180 degrees
- turned C29 to 180 degrees
- turned C30 to 180 degrees
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Routing:
- net +5V: track 445.6 -> 32.8 mm, vias 80 -> 0
- net /Row5: track 347.3 -> 38.5 mm
- net /Row2: track 346.1 -> 38.5 mm
- net /Row4: track 341.6 -> 38.5 mm
- net /Row3: track 250.7 -> 0.00 mm
- net Net-(LED50-DOUT): track 104.2 -> 0.00 mm
- net Net-(LED83-DIN): track 66.6 -> 0.00 mm
- net Net-(LED84-DIN): track 66.6 -> 0.00 mm
- net Net-(LED30-DIN): track 48.1 -> 0.00 mm
- net Net-(LED47-DOUT): track 42.8 -> 0.00 mm
- net Net-(LED88-DIN): track 40.4 -> 0.00 mm
- net Net-(LED13-DOUT): track 38.6 -> 0.00 mm
- net Net-(LED77-DOUT): track 38.0 -> 0.00 mm
- net Net-(LED16-DOUT): track 37.2 -> 0.00 mm
- net Net-(LED80-DOUT): track 27.7 -> 0.00 mm
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