File: keyboard-full/_restore_backup_2026-09-25T20-01-45-381/keyboard-full.kicad_sch (KiCad schematic)
At the start: 374 parts

Commit message: redid the keyboard pcb design
Connections:
- net +5V: no longer C48.1
- net Col0: now also A1.5 (GPIO3); no longer A1.2 (GPIO1)
- net Col1: now also A1.6 (GPIO4); no longer A1.4 (GPIO2)
- net Col10: now also A1.17 (GPIO13); no longer A1.16 (GPIO12)
- net Col11: now also A1.19 (GPIO14); no longer A1.17 (GPIO13)
- net Col12: now also A1.20 (GPIO15); no longer A1.19 (GPIO14)
- net Col13: now also A1.2 (GPIO1); no longer A1.20 (GPIO15)
- net Col2: now also A1.7 (GPIO5); no longer A1.5 (GPIO3)
- net Col3: now also A1.9 (GPIO6); no longer A1.6 (GPIO4)
- net Col4: now also A1.10 (GPIO7); no longer A1.7 (GPIO5)
- net Col5: now also A1.11 (GPIO8); no longer A1.9 (GPIO6)
- net Col6: now also A1.12 (GPIO9); no longer A1.10 (GPIO7)
- net Col7: now also A1.14 (GPIO10); no longer A1.11 (GPIO8)
- net Col8: now also A1.15 (GPIO11); no longer A1.14 (GPIO10)
- net Col9: now also A1.16 (GPIO12); no longer A1.15 (GPIO11)
- net LED: now also A1.1 (GPIO0); no longer A1.12 (GPIO9)
- net Row0: now also A1.4 (GPIO2); no longer A1.1 (GPIO0)
Other:
- moved on the sheet: C84
Changed lines of the file:
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@@
 	)
 	(junction
-		(at 270.51 337.82)
+		(at 269.24 337.82)
 		(diameter 0)
 		(color 0 0 0 0)
@@
 	)
 	(junction
-		(at 532.13 246.38)
-		(diameter 0)
-		(color 0 0 0 0)
-	)
-	(junction
 		(at 353.06 290.83)
 		(diameter 0)
@@
 	)
 	(junction
-		(at 270.51 322.58)
+		(at 269.24 322.58)
 		(diameter 0)
 		(color 0 0 0 0)
@@
 	(wire
 		(pts
-			(xy 270.51 336.55) (xy 270.51 337.82)
+			(xy 269.24 336.55) (xy 269.24 337.82)
 		)
 		(stroke
@@
 	(wire
 		(pts
-			(xy 532.13 246.38) (xy 532.13 252.73)
-		)
-		(stroke
-			(width 0)
-			(type default)
-		)
-	)
-	(wire
-		(pts
 			(xy 472.44 312.42) (xy 482.6 312.42)
 		)
@@
 	(wire
 		(pts
-			(xy 259.08 322.58) (xy 370.84 322.58)
+			(xy 259.08 322.58) (xy 269.24 322.58)
 		)
 		(stroke
@@
 	(wire
 		(pts
-			(xy 259.08 337.82) (xy 370.84 337.82)
+			(xy 259.08 337.82) (xy 269.24 337.82)
 		)
 		(stroke
@@
 	(wire
 		(pts
-			(xy 270.51 322.58) (xy 270.51 328.93)
+			(xy 269.24 322.58) (xy 269.24 328.93)
 		)
 		(stroke
@@
 	(wire
 		(pts
+			(xy 269.24 322.58) (xy 370.84 322.58)
+		)
+		(stroke
+			(width 0)
+			(type default)
+		)
+	)
+	(wire
+		(pts
 			(xy 175.26 236.22) (xy 185.42 236.22)
 		)
@@
 	(wire
 		(pts
+			(xy 269.24 337.82) (xy 370.84 337.82)
+		)
+		(stroke
+			(width 0)
+			(type default)
+		)
+	)
+	(wire
+		(pts
 			(xy 502.92 220.98) (xy 511.81 220.98)
 		)
@@
 	(wire
 		(pts
-			(xy 521.97 246.38) (xy 532.13 246.38)
+			(xy 521.97 246.38) (xy 549.91 246.38)
 		)
 		(stroke
@@
 	(wire
 		(pts
-			(xy 532.13 246.38) (xy 549.91 246.38)
-		)
-		(stroke
-			(width 0)
-			(type default)
-		)
-	)
-	(wire
-		(pts
 			(xy 109.22 261.62) (xy 119.38 261.62)
 		)
@@
 		)
 	)
-	(label "LED"
-		(at 25.4 246.38 0)
-		(effects
-			(font
-				(size 1.27 1.27)
-			)
-			(justify left bottom)
-		)
-	)
-	(label "Col12"
-		(at 25.4 259.08 0)
-		(effects
-			(font
-				(size 1.27 1.27)
-			)
-			(justify left bottom)
-		)
-	)
 	(label "Col7"
 		(at 154.94 167.64 0)
@@
 		)
 	)
-	(label "Col0"
-		(at 25.4 226.06 0)
+	(label "Col6"
+		(at 25.4 246.38 0)
 		(effects
 			(font
@@
 		)
 	)
-	(label "Col8"
-		(at 25.4 248.92 0)
+	(label "Col16"
+		(at 81.28 251.46 0)
 		(effects
 			(font
@@
 		)
 	)
-	(label "Col16"
-		(at 81.28 251.46 0)
+	(label "Col4"
+		(at 25.4 241.3 0)
 		(effects
 			(font
@@
 		)
 	)
-	(label "Col11"
-		(at 25.4 256.54 0)
+	(label "Col9"
+		(at 25.4 254 0)
 		(effects
 			(font
@@
 		)
 	)
-	(label "Col3"
-		(at 25.4 233.68 0)
+	(label "Col12"
+		(at 25.4 261.62 0)
 		(effects
 			(font
@@
 		)
 	)
+	(label "Col5"
+		(at 25.4 243.84 0)
+		(effects
+			(font
+				(size 1.27 1.27)
+			)
+			(justify left bottom)
+		)
+	)
 	(label "Row5"
 		(at 81.28 226.06 0)
@@
 		)
 	)
-	(label "Col1"
+	(label "Row0"
 		(at 25.4 228.6 0)
 		(effects
@@
 		)
 	)
+	(label "Col2"
+		(at 25.4 236.22 0)
+		(effects
+			(font
+				(size 1.27 1.27)
+			)
+			(justify left bottom)
+		)
+	)
+	(label "Col1"
+		(at 25.4 233.68 0)
+		(effects
+			(font
+				(size 1.27 1.27)
+			)
+			(justify left bottom)
+		)
+	)
 	(label "Col1"
 		(at 48.26 168.91 0)
@@
 		)
 	)
-	(label "Col7"
-		(at 25.4 243.84 0)
+	(label "Col8"
+		(at 25.4 251.46 0)
+		(effects
+			(font
+				(size 1.27 1.27)
+			)
+			(justify left bottom)
+		)
+	)
+	(label "Col13"
+		(at 25.4 226.06 0)
 		(effects
 			(font
@@
 		)
 	)
-	(label "Row3"
-		(at 337.82 106.68 0)
+	(label "Col0"
+		(at 25.4 231.14 0)
 		(effects
 			(font
@@
 		)
 	)
-	(label "Col10"
-		(at 25.4 254 0)
+	(label "Row3"
+		(at 337.82 106.68 0)
 		(effects
 			(font
@@
 		)
 	)
-	(label "Row0"
-		(at 337.82 39.37 0)
+	(label "Col10"
+		(at 25.4 256.54 0)
 		(effects
 			(font
@@
 		)
 	)
-	(label "Col9"
-		(at 25.4 251.46 0)
+	(label "Row0"
+		(at 337.82 39.37 0)
 		(effects
 			(font
@@
 		)
 	)
-	(label "Col2"
-		(at 25.4 231.14 0)
-		(effects
-			(font
-				(size 1.27 1.27)
-			)
-			(justify left bottom)
-		)
-	)
 	(label "Col6"
 		(at 137.16 167.64 0)
@@
 		)
 	)
-	(label "Col5"
-		(at 25.4 238.76 0)
+	(label "LED"
+		(at 25.4 223.52 0)
 		(effects
 			(font
@@
 		)
 	)
-	(label "Row0"
-		(at 25.4 223.52 0)
+	(label "Row2"
+		(at 81.28 233.68 0)
 		(effects
 			(font
@@
 		)
 	)
-	(label "Row2"
-		(at 81.28 233.68 0)
+	(label "Col7"
+		(at 25.4 248.92 0)
 		(effects
 			(font
@@
 		)
 	)
-	(label "Row4"
-		(at 81.28 228.6 0)
-		(effects
-			(font
-				(size 1.27 1.27)
-			)
-			(justify left bottom)
-		)
-	)
-	(label "Col14"
-		(at 81.28 256.54 0)
+	(label "Col3"
+		(at 25.4 238.76 0)
 		(effects
 			(font
@@
 		)
 	)
-	(label "Col4"
-		(at 25.4 236.22 0)
+	(label "Row4"
+		(at 81.28 228.6 0)
 		(effects
 			(font
@@
 		)
 	)
-	(label "Col13"
-		(at 25.4 261.62 0)
+	(label "Col14"
+		(at 81.28 256.54 0)
 		(effects
 			(font
@@
 		)
 	)
-	(label "Col6"
-		(at 25.4 241.3 0)
+	(label "Col11"
+		(at 25.4 259.08 0)
 		(effects
 			(font
@@
 	(symbol
 		(lib_id "Device:C")
-		(at 270.51 332.74 0)
+		(at 269.24 332.74 0)
 		(unit 1)
 		(body_style 1)
@@
 		(dnp no)
 		(property "Reference" "C84"
-			(at 273.05 331.724 0)
+			(at 271.78 331.724 0)
 			(show_name no)
 			(do_not_autoplace no)
@@
 		)
 		(property "Value" "0.1uF"
-			(at 273.05 334.264 0)
+			(at 271.78 334.264 0)
 			(show_name no)
 			(do_not_autoplace no)
@@
 		)
 		(property "Footprint" "Capacitor_SMD:C_1206_3216Metric_Pad1.33x1.80mm_HandSolder"
-			(at 271.4752 336.55 0)
+			(at 270.2052 336.55 0)
 			(hide yes)
 			(show_name no)
@@
 		)
 		(property "Datasheet" ""
-			(at 270.51 332.74 0)
+			(at 269.24 332.74 0)
 			(hide yes)
 			(show_name no)
@@
 		)
 		(property "Description" "Unpolarized capacitor"
-			(at 270.51 332.74 0)
+			(at 269.24 332.74 0)
 			(hide yes)
 			(show_name no)
